File: kicad/PROMProgrammer.kicad_pcb (KiCad board)
At the start: 2 copper layers, 174.5 x 93 mm, 97 parts, among them J1 Control / Program Select Swit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, J2 USB_C_Receptacle_PowerOnly_6P, J3 Conn_01x02, J4 USB_A, J5 Barrel_Jack, Q2 2N3904, Q3 2N3904, Q4 BD139, Q5 2N3904, Q6 2N3904, SW1 SW_SPDT, SW11 SW_Push_SPDT, SW12 SW_Push_SPDT, SW13 SW_Push_SPDT, SW14 SW_Push_SPDT, SW15 SW_Push_SPDT, SW16 SW_Push_SPDT, SW17 SW_Push_SPDT, SW18 SW_Push_SPDT, SW2 SW_SPDT, SW3 SW_SPDT, SW4 SW_SPDT, SW5 SW_SPDT, SW6 SW_SPDT, SW8 SW_SPDT, U1 74S188, U2 MC34063AP, U6 4043, U7 4017, U8 HEF4093B, U9 TL431LP

Commit message: All working and tidy
Other:
- board text added: "49fe3df8-a061-4c38-bd2d-84204057c43a"
- board text removed: "748009cc-844e-416f-8f3c-c4b696d091e6"
Changed lines of the file:
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@@
 	(title_block
 		(title "PROM Programmer -Transistor Update")
-		(date "2025-08-08")
+		(date "2025-08-22")
 		(rev "3.1")
 	)
@@
 		)
 	)
-	(gr_text "748009cc-844e-416f-8f3c-c4b696d091e6 "
+	(gr_text "49fe3df8-a061-4c38-bd2d-84204057c43a"
 		(at 183.03869 147.216126 0)
 		(layer "F.SilkS")
